Commit message: restrcutred repo

File: dog_walking/resources/dog.urdf (robot description, URDF)
Before this commit: robot materials, 17 links, 16 joints
Links:
- link coxa_BL: mass 0.09 -> 0.2
- link coxa_BR: mass 0.09 -> 0.2
- link coxa_FL: mass 0.075 -> 0.3
- link coxa_FR: mass 0.075 -> 0.3
- link femur_BL: mass 0.085 -> 0.3
- link femur_BR: mass 0.085 -> 0.3
- link femur_FL: mass 0.084 -> 0.3
- link femur_FR: mass 0.084 -> 0.3
- link foot_BL: mass 0.0044 -> 0.15
- link foot_BR: mass 0.0044 -> 0.15
- link foot_FL: mass 0.0044 -> 0.15
- link foot_FR: mass 0.0044 -> 0.15
- link tibia_BL: mass 0.034 -> 0.15
- link tibia_BR: mass 0.034 -> 0.15
- link tibia_FL: mass 0.034 -> 0.15
- link tibia_FR: mass 0.034 -> 0.15
